File: maclock-pcb/maclock-breakout.kicad_sch (KiCad schematic)
At the start: 0 parts

Commit message: updated board design to 2026.5
Parts:
- added BAT+: 5V, symbol Connector_Generic:Conn_01x01
- added BAT-: GND, symbol Connector_Generic:Conn_01x01
- added C1: 100nF, Capacitor_THT:C_Disc_D6.0mm_W2.5mm_P5.00mm, symbol Device:C
- added JP1: Rotary_Encoder_5pin, KiCad:1X05_ROUND_70, symbol Device:RotaryEncoder_Switch
- added PiInput: PiInput, Connector_PinHeader_2.54mm:PinHeader_1x07_P2.54mm_Vertical, symbol Connector_Generic:Conn_01x07
- added R1, R2, R3: 1K, Resistor_SMD:R_0402_1005Metric_Pad0.72x0.64mm_HandSolder, symbol Device:R
- added SW1, SW2: SW_Push, KiCad:TS32735BK160RASMTTR, symbol Switch:SW_Push
Connections:
- new net 5V: BAT+.1 (Pin_1), PiInput.4 (Pin_4), R1.1, R2.1, R3.1
- new net AUDIO: C1.1, PiInput.5 (Pin_5)
- new net BTN1: PiInput.7 (Pin_7), R1.2, SW1.1
- new net BTN2: PiInput.6 (Pin_6), R2.2, SW2.1
- new net ENC_A: JP1.A, PiInput.3 (Pin_3)
- new net ENC_B: JP1.B, PiInput.1 (Pin_1)
- new net ENC_SW: JP1.S1, R3.2
- new net GND: BAT-.1 (Pin_1), C1.2, JP1.C, JP1.S2, PiInput.2 (Pin_2), SW1.2, SW2.2
Other:
- note added: "Maclock breakout — connects Pi Zero 2W GPIO to front-panel parts (encoder, 2 buttons, audio to PAM8302, speaker)"
- note added: "Net → Pi pin: 5V→2, GND→6, BTN1→13, ENC_B→19, ENC_A→23, AUDIO→35, BTN2→37"
- note added: "Note: schematic captures design intent based on the maclock-build wiring guide. R3 placement (encoder push-switch pull-up) and C1 topology (decoupling-to-GND) are assumed; verify against PCB if used for a board revision."
Changed lines of the file:
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@@
-(kicad_sch
-	(version 20250114)
-	(generator "eeschema")
-	(generator_version "9.0")
-	(paper "A4")
-	(sheet_instances
-		(path "/"
-			(page "1")
-		)
-	)
-	(embedded_fonts no)
-)
