File: maclock-pcb/maclock-breakout.kicad_sch (KiCad schematic)
At the start: 25 parts, among them J1 53398-0271, J2 53398-0471, J3 53398-0271, J4 Pi GPIO, SW1 TSB001A3518A, SW2 TSB001A3518A, U1 PAM8302AASCR, U2 SN74LVC1G17DBVR, U3 TPS7A2030PDBVR

Commit message: Revert "Breakout: ENC1 is an Alps EC05E1220401 over a shaft cutout"
This reverts commit d02c471. The test Alps was loose on the dial too, so
ENC1 is back on the F-Switch E8E8 footprint, the one encoder known to fit,
and J1-J3 are back where they were. PCBway buys only from LCSC, DigiKey and
Mouser, so the board goes to assembly with ENC1 left off and the E8E8 is
hand-soldered; the README says so.
Parts:
- ENC1: value EC05E1220401 -> E8E8-3.2C60-9B34; footprint maclock:RotaryEncoder_Alps_EC05E1220401_SMD -> maclock:RotaryEncoder_E8E8-3.2C60-9B34_SMD; LCSC C116648 -> (none); MPN EC05E1220401 -> E8E8-3.2C60-9B34; Manufacturer Alps Alpine -> F-Switch; Supplier (none) -> dicomon; Supplier Link (none) -> https://www.dicomon.com/index.php?ctl=Product&met=detail&it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
Changed lines of the file:
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@@
 			)
 		)
-		(property "Value" "EC05E1220401"
+		(property "Value" "E8E8-3.2C60-9B34"
 			(at 140.97 107.95 0)
 			(show_name no)
@@
 			)
 		)
-		(property "Footprint" "maclock:RotaryEncoder_Alps_EC05E1220401_SMD"
+		(property "Footprint" "maclock:RotaryEncoder_E8E8-3.2C60-9B34_SMD"
 			(at 134.62 101.6 0)
 			(hide yes)
@@
 			)
 		)
-		(property "Datasheet" "https://tech.alpsalpine.com/assets/catalog/product-catalog-ec-all.en.pdf"
+		(property "Datasheet" "https://www.dicomon.com/index.php?ctl=Product&met=detail&item_id=1037"
 			(at 134.62 101.6 0)
 			(hide yes)
@@
 			)
 		)
-		(property "Description" "Alps Alpine EC05E1220401 5 mm hollow-shaft encoder, vertical SMD, 12 pulse / 12 detent, 1.72 mm hex hole; MP = the frame's solder tabs"
+		(property "Description" "F-Switch E8E8-3.2C60-9B34 SMD mouse-wheel encoder, 9 pulse / 18 detent, 1.74 mm hex bore; MP = the cover's solder tabs"
 			(at 134.62 101.6 0)
 			(hide yes)
@@
 			)
 		)
-		(property "Manufacturer" "Alps Alpine"
+		(property "Manufacturer" "F-Switch"
 			(at 134.62 101.6 0)
 			(hide yes)
@@
 			)
 		)
-		(property "MPN" "EC05E1220401"
+		(property "MPN" "E8E8-3.2C60-9B34"
 			(at 134.62 101.6 0)
 			(hide yes)
@@
 			)
 		)
-		(property "LCSC" "C116648"
+		(property "LCSC" ""
 			(at 134.62 101.6 0)
 			(hide yes)
@@
 			)
 		)
-		(property "Supplier" ""
+		(property "Supplier" "dicomon"
 			(at 134.62 101.6 0)
 			(hide yes)
@@
 			)
 		)
-		(property "Supplier Link" ""
+		(property "Supplier Link" "https://www.dicomon.com/index.php?ctl=Product&met=detail&item_id=1037"
 			(at 134.62 101.6 0)
 			(hide yes)

Commit message: Breakout: ENC1 is a TT EN10HT lying flat, pins west
PCBway can't buy the E8E8, and every vertical SMD encoder at LCSC, DigiKey
and Mouser has a bore that is too loose or too short for the dial. Mouse-wheel
encoders laid on their back do fit: the bore is 1.74 mm and the 5 mm-thick
body reaches the full-width part of the dial's tapered shaft. TT Electronics'
EN10HT is that kind of encoder built to lie flat with the bore up, so it goes
in like any through-hole part, and DigiKey stocks it. Its 1.75 +/-0.03 mm
bore is untested on the dial; the top of that range is looser than the TTC
part that fits.

- maclock:RotaryEncoder_EN10HT1212N5HH3_THT, origin on the bore at the old
  ENC1 spot. Land from TT's EN10 datasheet, placed on the bore with TT's
  STEP: pin holes 6.8 mm west of the bore (TT dimensions them 5.5 mm from the
  tab line, which sits 1.3 mm off the bore) and an oval slot for the north
  bracket tab. The south tab falls past the board edge. The pads run 2.6 mm
  east of the holes so a laid-flat Huano 4.5 or HOAUC HYCW04 can be
  lap-soldered instead. TT's STEP is the 3D model. E8E8 footprint and model
  removed.
- Pins west keep the holes clear of the bottom-side parts. The north tab's
  slot landed on U3 and C8, so U3 moves 4.4 mm west and C8 4.3 mm west;
  +5V reaches C8 round the slot's north side and U3's EN tie goes round its
  south side. U3's +3V0 and GND are redrawn to match. Three GND stitching
  vias move off the new pads and the new ENC_B route.
- ENC_A and ENC_B re-routed on F.Cu to the new pads.
- Symbol renamed maclock:RotaryEncoder_EN10HT1212N5HH3 with TT and DigiKey
  fields; the schematic note says the same. J3's Speaker label and U3's
  reference moved clear of the new pads and the board edge.

DRC as before (one text-thickness warning), 0 unconnected, schematic parity
clean, ERC 0.
Parts:
- ENC1: value E8E8-3.2C60-9B34 -> EN10HT1212N5HH3; footprint maclock:RotaryEncoder_E8E8-3.2C60-9B34_SMD -> maclock:RotaryEncoder_EN10HT1212N5HH3_THT; symbol maclock:RotaryEncoder_E8E8-3.2C60-9B34 -> maclock:RotaryEncoder_EN10HT1212N5HH3; MPN E8E8-3.2C60-9B34 -> EN10HT1212N5HH3; Manufacturer F-Switch -> TT Electronics; Supplier dicomon -> DigiKey; Supplier Link https://www.dicomon.com/index.php?ctl=Product&met=detail&it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 -> https://www.digikey.com/en/products/detail/tt-electronics-b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
Other:
- note added: "TT Electronics EN10HT1212N5HH3 from DigiKey (lies flat, bore up; not stocked at LCSC). C is the common pin. The Pi enables internal pull-ups on GPIO 11 (A) and GPIO 10 (B)."
- note removed: "F-Switch E8E8-3.2C60-9B34 from dicomon (item 1037; not stocked at LCSC). C is the common pin. The Pi enables internal pull-ups on GPIO 11 (A) and GPIO 10 (B)."
Changed lines of the file:
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@@
 		)
 	)
-	(text "F-Switch E8E8-3.2C60-9B34 from dicomon\n(item 1037; not stocked at LCSC).\nC is the common pin. The Pi enables internal\npull-ups on GPIO 11 (A) and GPIO 10 (B)."
+	(text "TT Electronics EN10HT1212N5HH3 from DigiKey\n(lies flat, bore up; not stocked at LCSC).\nC is the common pin. The Pi enables internal\npull-ups on GPIO 11 (A) and GPIO 10 (B)."
 		(exclude_from_sim no)
 		(at 101.6 121.92 0)
@@
 	)
 	(symbol
-		(lib_id "maclock:RotaryEncoder_E8E8-3.2C60-9B34")
+		(lib_id "maclock:RotaryEncoder_EN10HT1212N5HH3")
 		(at 134.62 101.6 0)
 		(unit 1)
@@
 			)
 		)
-		(property "Value" "E8E8-3.2C60-9B34"
+		(property "Value" "EN10HT1212N5HH3"
 			(at 140.97 107.95 0)
 			(show_name no)
@@
 			)
 		)
-		(property "Footprint" "maclock:RotaryEncoder_E8E8-3.2C60-9B34_SMD"
+		(property "Footprint" "maclock:RotaryEncoder_EN10HT1212N5HH3_THT"
 			(at 134.62 101.6 0)
 			(hide yes)
@@
 			)
 		)
-		(property "Datasheet" "https://www.dicomon.com/index.php?ctl=Product&met=detail&item_id=1037"
+		(property "Datasheet" "https://www.ttelectronics.com/TTElectronics/media/ProductFiles/Datasheet/EN10.pdf"
 			(at 134.62 101.6 0)
 			(hide yes)
@@
 			)
 		)
-		(property "Description" "F-Switch E8E8-3.2C60-9B34 SMD mouse-wheel encoder, 9 pulse / 18 detent, 1.74 mm hex bore; MP = the cover's solder tabs"
+		(property "Description" "TT Electronics EN10HT1212N5HH3 top-adjust 10 mm encoder, lies flat with the hex bore up, 12 pulse / 12 detent, 1.75 mm hex bore; MP = the bracket tab"
 			(at 134.62 101.6 0)
 			(hide yes)
@@
 			)
 		)
-		(property "Manufacturer" "F-Switch"
+		(property "Manufacturer" "TT Electronics"
 			(at 134.62 101.6 0)
 			(hide yes)
@@
 			)
 		)
-		(property "MPN" "E8E8-3.2C60-9B34"
+		(property "MPN" "EN10HT1212N5HH3"
 			(at 134.62 101.6 0)
 			(hide yes)
@@
 			)
 		)
-		(property "Supplier" "dicomon"
+		(property "Supplier" "DigiKey"
 			(at 134.62 101.6 0)
 			(hide yes)
@@
 			)
 		)
-		(property "Supplier Link" "https://www.dicomon.com/index.php?ctl=Product&met=detail&item_id=1037"
+		(property "Supplier Link" "https://www.digikey.com/en/products/detail/tt-electronics-bi/EN10HT1212N5HH3/16360755"
 			(at 134.62 101.6 0)
 			(hide yes)

Commit message: Revert "Breakout: ENC1 is a TT EN10HT lying flat, pins west"
This reverts commit 263cf97165d9f075fd2916f10ce5fd05847f6fb2.
Parts:
- ENC1: value EN10HT1212N5HH3 -> E8E8-3.2C60-9B34; footprint maclock:RotaryEncoder_EN10HT1212N5HH3_THT -> maclock:RotaryEncoder_E8E8-3.2C60-9B34_SMD; symbol maclock:RotaryEncoder_EN10HT1212N5HH3 -> maclock:RotaryEncoder_E8E8-3.2C60-9B34; MPN EN10HT1212N5HH3 -> E8E8-3.2C60-9B34; Manufacturer TT Electronics -> F-Switch; Supplier DigiKey -> dicomon; Supplier Link https://www.digikey.com/en/products/detail/tt-electronics-b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 -> https://www.dicomon.com/index.php?ctl=Product&met=detail&it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
Other:
- note added: "F-Switch E8E8-3.2C60-9B34 from dicomon (item 1037; not stocked at LCSC). C is the common pin. The Pi enables internal pull-ups on GPIO 11 (A) and GPIO 10 (B)."
- note removed: "TT Electronics EN10HT1212N5HH3 from DigiKey (lies flat, bore up; not stocked at LCSC). C is the common pin. The Pi enables internal pull-ups on GPIO 11 (A) and GPIO 10 (B)."
Changed lines of the file:
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@@
 		)
 	)
-	(text "TT Electronics EN10HT1212N5HH3 from DigiKey\n(lies flat, bore up; not stocked at LCSC).\nC is the common pin. The Pi enables internal\npull-ups on GPIO 11 (A) and GPIO 10 (B)."
+	(text "F-Switch E8E8-3.2C60-9B34 from dicomon\n(item 1037; not stocked at LCSC).\nC is the common pin. The Pi enables internal\npull-ups on GPIO 11 (A) and GPIO 10 (B)."
 		(exclude_from_sim no)
 		(at 101.6 121.92 0)
@@
 	)
 	(symbol
-		(lib_id "maclock:RotaryEncoder_EN10HT1212N5HH3")
+		(lib_id "maclock:RotaryEncoder_E8E8-3.2C60-9B34")
 		(at 134.62 101.6 0)
 		(unit 1)
@@
 			)
 		)
-		(property "Value" "EN10HT1212N5HH3"
+		(property "Value" "E8E8-3.2C60-9B34"
 			(at 140.97 107.95 0)
 			(show_name no)
@@
 			)
 		)
-		(property "Footprint" "maclock:RotaryEncoder_EN10HT1212N5HH3_THT"
+		(property "Footprint" "maclock:RotaryEncoder_E8E8-3.2C60-9B34_SMD"
 			(at 134.62 101.6 0)
 			(hide yes)
@@
 			)
 		)
-		(property "Datasheet" "https://www.ttelectronics.com/TTElectronics/media/ProductFiles/Datasheet/EN10.pdf"
+		(property "Datasheet" "https://www.dicomon.com/index.php?ctl=Product&met=detail&item_id=1037"
 			(at 134.62 101.6 0)
 			(hide yes)
@@
 			)
 		)
-		(property "Description" "TT Electronics EN10HT1212N5HH3 top-adjust 10 mm encoder, lies flat with the hex bore up, 12 pulse / 12 detent, 1.75 mm hex bore; MP = the bracket tab"
+		(property "Description" "F-Switch E8E8-3.2C60-9B34 SMD mouse-wheel encoder, 9 pulse / 18 detent, 1.74 mm hex bore; MP = the cover's solder tabs"
 			(at 134.62 101.6 0)
 			(hide yes)
@@
 			)
 		)
-		(property "Manufacturer" "TT Electronics"
+		(property "Manufacturer" "F-Switch"
 			(at 134.62 101.6 0)
 			(hide yes)
@@
 			)
 		)
-		(property "MPN" "EN10HT1212N5HH3"
+		(property "MPN" "E8E8-3.2C60-9B34"
 			(at 134.62 101.6 0)
 			(hide yes)
@@
 			)
 		)
-		(property "Supplier" "DigiKey"
+		(property "Supplier" "dicomon"
 			(at 134.62 101.6 0)
 			(hide yes)
@@
 			)
 		)
-		(property "Supplier Link" "https://www.digikey.com/en/products/detail/tt-electronics-bi/EN10HT1212N5HH3/16360755"
+		(property "Supplier Link" "https://www.dicomon.com/index.php?ctl=Product&met=detail&item_id=1037"
 			(at 134.62 101.6 0)
 			(hide yes)

Commit message: Breakout: ENC1 is a HUANO 4.5 laid flat, pins north, fitted by hand
No vertical encoder at LCSC, DigiKey or Mouser grips the dial: the bores
are too loose or too short. A HUANO 4.5 mm mouse-wheel encoder laid on its
back does: its 1.74 mm bore and 5 mm-thick body reach the full-width part of
the dial's tapered shaft. Nothing like it is sold where PCBway buys, so ENC1
is fitted by hand.

- maclock:RotaryEncoder_HUANO_4.5mm_LayFlat_SMD, origin on the bore at the
  old ENC1 spot, pins pointing north. Top-side pads at 2.5 mm pitch for the
  pins, bent down, plus two MP pads for the frame's clip legs. HUANO
  publishes no drawing, so the pads run 2.8 mm north from just outside the
  body (estimated from the listing photo) to catch the pins wherever they
  land. No paste, thermal reliefs on the GND pads, no 3D model. E8E8
  footprint and model removed.
- Pin order assumed C-B-A with the common at one end, as on HOAUC's and
  TT's mouse-wheel encoders: C (west pad) = GND, B = ENC_B, A = ENC_A.
  Turning the part face-down swaps the two ends.
- ENC_A and ENC_B re-routed on F.Cu to the new pads; nothing else moves.
- ENC1 is out of the BOM and placement files (not DNP: it is fitted, just
  not by PCBway). Symbol renamed maclock:RotaryEncoder_HUANO_4.5mm, with
  Amazon as the supplier; the schematic note and README say how to fit it.

DRC as before (one text-thickness warning), 0 unconnected, schematic parity
clean, ERC 0.
Parts:
- ENC1: value E8E8-3.2C60-9B34 -> HUANO 4.5; footprint maclock:RotaryEncoder_E8E8-3.2C60-9B34_SMD -> maclock:RotaryEncoder_HUANO_4.5mm_LayFlat_SMD; symbol maclock:RotaryEncoder_E8E8-3.2C60-9B34 -> maclock:RotaryEncoder_HUANO_4.5mm; MPN E8E8-3.2C60-9B34 -> (none); Manufacturer F-Switch -> HUANO; Supplier dicomon -> Amazon; Supplier Link https://www.dicomon.com/index.php?ctl=Product&met=detail&it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 -> https://www.amazon.com/dp/B0C13ZZVT5; now left out of the parts list
Other:
- note added: "HUANO 4.5 mm mouse-wheel encoder, laid on its back (fitted by hand, left out of the PCBway BOM). C is the common pin. The Pi enables internal pull-ups on GPIO 11 (A) and GPIO 10 (B)."
- note removed: "F-Switch E8E8-3.2C60-9B34 from dicomon (item 1037; not stocked at LCSC). C is the common pin. The Pi enables internal pull-ups on GPIO 11 (A) and GPIO 10 (B)."
Changed lines of the file:
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@@
 		)
 	)
-	(text "F-Switch E8E8-3.2C60-9B34 from dicomon\n(item 1037; not stocked at LCSC).\nC is the common pin. The Pi enables internal\npull-ups on GPIO 11 (A) and GPIO 10 (B)."
+	(text "HUANO 4.5 mm mouse-wheel encoder, laid on its back\n(fitted by hand, left out of the PCBway BOM).\nC is the common pin. The Pi enables internal\npull-ups on GPIO 11 (A) and GPIO 10 (B)."
 		(exclude_from_sim no)
 		(at 101.6 121.92 0)
@@
 	)
 	(symbol
-		(lib_id "maclock:RotaryEncoder_E8E8-3.2C60-9B34")
+		(lib_id "maclock:RotaryEncoder_HUANO_4.5mm")
 		(at 134.62 101.6 0)
 		(unit 1)
 		(body_style 1)
 		(exclude_from_sim no)
-		(in_bom yes)
+		(in_bom no)
 		(on_board yes)
-		(in_pos_files yes)
+		(in_pos_files no)
 		(dnp no)
 		(property "Reference" "ENC1"
@@
 			)
 		)
-		(property "Value" "E8E8-3.2C60-9B34"
+		(property "Value" "HUANO 4.5"
 			(at 140.97 107.95 0)
 			(show_name no)
@@
 			)
 		)
-		(property "Footprint" "maclock:RotaryEncoder_E8E8-3.2C60-9B34_SMD"
+		(property "Footprint" "maclock:RotaryEncoder_HUANO_4.5mm_LayFlat_SMD"
 			(at 134.62 101.6 0)
 			(hide yes)
@@
 			)
 		)
-		(property "Datasheet" "https://www.dicomon.com/index.php?ctl=Product&met=detail&item_id=1037"
+		(property "Datasheet" ""
 			(at 134.62 101.6 0)
 			(hide yes)
@@
 			)
 		)
-		(property "Description" "F-Switch E8E8-3.2C60-9B34 SMD mouse-wheel encoder, 9 pulse / 18 detent, 1.74 mm hex bore; MP = the cover's solder tabs"
+		(property "Description" "HUANO 4.5 mm mouse-wheel encoder laid on its back, 1.74 mm hex bore up, legs bent down onto top-side pads; MP = the frame's clip legs. Hand-fitted"
 			(at 134.62 101.6 0)
 			(hide yes)
@@
 			)
 		)
-		(property "Manufacturer" "F-Switch"
+		(property "Manufacturer" "HUANO"
 			(at 134.62 101.6 0)
 			(hide yes)
@@
 			)
 		)
-		(property "MPN" "E8E8-3.2C60-9B34"
+		(property "MPN" ""
 			(at 134.62 101.6 0)
 			(hide yes)
@@
 			)
 		)
-		(property "Supplier" "dicomon"
+		(property "Supplier" "Amazon"
 			(at 134.62 101.6 0)
 			(hide yes)
@@
 			)
 		)
-		(property "Supplier Link" "https://www.dicomon.com/index.php?ctl=Product&met=detail&item_id=1037"
+		(property "Supplier Link" "https://www.amazon.com/dp/B0C13ZZVT5"
 			(at 134.62 101.6 0)
 			(hide yes)
